Commit message: phase 1 simulation done

File: src/waymaster_v1/description/robotv1.urdf (robot description, URDF)
Before this commit: robot waymasterv1, 5 links, 4 joints
Links:
- added link left_motor, mass 0.2; collision box size=0.06 0.035 0.040; visual box size=0.06 0.035 0.040
- added link right_motor, mass 0.2; collision box size=0.06 0.035 0.040; visual box size=0.06 0.035 0.040
- link castor_wheel: mass None -> 0.1
- link chassis: mass None -> 0.5; geometry collision box size=0.3 0.23 0.15; visual box size=0.3 0.23 0.15
- link left_wheel: mass None -> 0.1
- link right_wheel: mass None -> 0.1
Joints:
- added joint left_motor_joint: type fixed, parent base_link, child left_motor, origin xyz=0.0 0.09 0.0515 rpy=0.0 0.0 1.571
- added joint right_motor_joint: type fixed, parent base_link, child right_motor, origin xyz=0.0 -0.09 0.0515 rpy=0.0 0.0 -1.571
- joint castor_wheel_joint: origin xyz=0.24 0.0 0.0 rpy=0.0 0.0 0.0 -> xyz=0.24 0.0 0.0515 rpy=0.0 0.0 0.0
- joint left_wheel_joint: origin xyz=0.0 0.175 0.0 rpy=-1.571 0.0 0.0 -> xyz=0.0 0.14 0.0515 rpy=-1.571 0.0 0.0
- joint right_wheel_joint: origin xyz=0.0 -0.175 0.0 rpy=1.571 0.0 0.0 -> xyz=0.0 -0.14 0.0515 rpy=1.571 0.0 0.0

Commit message: added new launch, world and arduino files

File: src/waymaster_v1/description/robotv1.urdf (robot description, URDF)
Before this commit: robot waymasterv1, 7 links, 6 joints
Links:
- added link laser_frame, mass 0.1; collision cylinder length=0.04 radius=0.05; visual cylinder length=0.04 radius=0.05
Joints:
- added joint laser_joint: type fixed, parent chassis, child laser_frame, origin xyz=0.122 0 0.212 rpy=0 0 0

Commit message: added cmd_vel to arduino

File: src/waymaster_v1/description/robotv1.urdf (robot description, URDF)
Before this commit: robot waymasterv1, 8 links, 7 joints
Joints:
- removed joint left_wheel_joint
- removed joint right_wheel_joint
- added joint wheel_left_joint: type continuous, parent base_link, child left_wheel, origin xyz=0.0 0.14 0.0515 rpy=-1.571 0.0 0.0, axis 0.0 0.0 1.0
- added joint wheel_right_joint: type continuous, parent base_link, child right_wheel, origin xyz=0.0 -0.14 0.0515 rpy=1.571 0.0 0.0, axis 0.0 0.0 -1.0

Commit message: ros to ard and ard to ros nav stack complete.

File: src/waymaster_v1/description/robotv1.urdf (robot description, URDF)
Before this commit: robot waymasterv1, 8 links, 7 joints
Links:
- removed link laser_frame
- removed link left_motor
- removed link right_motor
- added link base_footprint
- added link camera_link, mass 0.1; collision cylinder length=0.04 radius=0.05; visual cylinder length=0.04 radius=0.05
Joints:
- removed joint laser_joint
- removed joint left_motor_joint
- removed joint right_motor_joint
- removed joint wheel_left_joint
- removed joint wheel_right_joint
- added joint base_footprint_joint: type fixed, parent base_link, child base_footprint, origin xyz=0.0 0.0 0.0 rpy=0.0 0.0 0.0
- added joint camera_joint: type fixed, parent chassis, child camera_link, origin xyz=0.122 0 0.212 rpy=0 0 0
- added joint left_wheel_joint: type continuous, parent base_link, child left_wheel, origin xyz=0.0 0.14 0.0515 rpy=-1.571 0.0 0.0, axis 0.0 0.0 1.0
- added joint right_wheel_joint: type continuous, parent base_link, child right_wheel, origin xyz=0.0 -0.14 0.0515 rpy=1.571 0.0 0.0, axis 0.0 0.0 -1.0
